File: i-fucking-love-fucking-you.kicad_sch (KiCad schematic)
At the start: 65 parts, among them J1 Conn_01x06_Female, J2 Conn_01x05_Male, Q1 2N7000, Q2 2N7000, U1 ATtiny10-TS

Commit message: added code to do rand from adc on start
Parts:
- removed Q1, Q2: 2N7000, Package_TO_SOT_SMD:SOT-23, symbol Transistor_FET:2N7000
- added Q1, Q2: MMDT2222A, Package_TO_SOT_SMD:SOT-23, symbol Transistor_BJT:MMDT2222A
- added R3, R5: 1K Ohm, Resistor_SMD:R_0603_1608Metric_Pad0.98x0.95mm_HandSolder, symbol Device:R_Small
- C1: value C_Small -> .1uF
- R1, R2: value R_Small -> 68 Ohm
- R4: renamed from R3; value R_Small -> 68 Ohm
Connections:
- net GND: now also Q1.1 (E2), Q2.1 (E2)
- net at R4.1: now also Q2.3 (C2)
- net at U1.4 (PB2): now also R5.2
- net at R2.1: now also Q1.3 (C2)
- net at J2.3 (Pin_3), U1.3 (PB1): now also R3.1
- new net: Q2.2 (B2), R5.1
- new net: Q1.2 (B2), R3.2
